Commit message: Feedback from hardware and visualization of robot in rviz2 in real time - Added a node for simulated hardware feedback in case don't have it - Added some params for collisions - Virtual moveit controller for flippers - Can you move and visualizer the flippers

File: workspace/src/robot_moveit_config/config/rescue_robot.ros2_control.xacro (robot description, xacro)
@@ -6,5 +6,5 @@
             <hardware>
                 <!-- By default, set up controllers for simulation. This won't work on real hardware -->
-                <plugin>mock_components/GenericSystem</plugin>
+                <plugin>aesir_plugin/TopicBridgeHardware</plugin>
             </hardware>
             <joint name="joint_1">
@@ -68,4 +68,28 @@
                 <state_interface name="effort"/>
             </joint>
+            <joint name="flipper_1_joint">
+                <command_interface name="position"/>
+                <state_interface name="position">
+                    <param name="initial_value">${initial_positions['flipper_1_joint']}</param>
+                </state_interface>
+            </joint>
+            <joint name="flipper_2_joint">
+                <command_interface name="position"/>
+                <state_interface name="position">
+                    <param name="initial_value">${initial_positions['flipper_2_joint']}</param>
+                </state_interface>
+            </joint>
+            <joint name="flipper_3_joint">
+                <command_interface name="position"/>
+                <state_interface name="position">
+                    <param name="initial_value">${initial_positions['flipper_3_joint']}</param>
+                </state_interface>
+            </joint>
+            <joint name="flipper_4_joint">
+                <command_interface name="position"/>
+                <state_interface name="position">
+                    <param name="initial_value">${initial_positions['flipper_4_joint']}</param>
+                </state_interface>
+            </joint>
         </ros2_control>
     </xacro:macro>
