Commit message: Fix bugs and new launch - Divided the bringup in with rviz2, and without it - Fix bug of hardware plugin sending flippers commands

File: workspace/src/aesir_robot_description/urdf/rescue_robot.urdf.xacro (robot description, xacro)
@@ -44,5 +44,5 @@
       <origin rpy="0 0 0" xyz="0 0.757 0"/>
       <geometry>
-        <mesh filename="file://$(find aesir_robot_description)/meshes/base.stl" scale="0.001 0.001 0.001"/>
+        <mesh filename="package://aesir_robot_description/meshes/base.stl" scale="0.001 0.001 0.001"/>
       </geometry>
     </visual>
@@ -50,5 +50,5 @@
       <origin rpy="0 0 0" xyz="0 0.757 0."/>
       <geometry>
-        <mesh filename="file://$(find aesir_robot_description)/meshes/base.stl" scale="0.001 0.001 0.001"/>
+        <mesh filename="package://aesir_robot_description/meshes/base.stl" scale="0.001 0.001 0.001"/>
       </geometry>
     </collision>
@@ -63,9 +63,9 @@
     <visual>
       <origin rpy="0 0 0" xyz="0.3 1.06 0"/>
-      <geometry><mesh filename="file://$(find aesir_robot_description)/meshes/flipper_1.stl" scale="0.001 0.001 0.001"/></geometry>
+      <geometry><mesh filename="package://aesir_robot_description/meshes/flipper_1.stl" scale="0.001 0.001 0.001"/></geometry>
     </visual>
     <collision>
       <origin rpy="0 0 0" xyz="0.3 1.06 0"/>
-      <geometry><mesh filename="file://$(find aesir_robot_description)/meshes/flipper_1.stl" scale="0.001 0.001 0.001"/></geometry>
+      <geometry><mesh filename="package://aesir_robot_description/meshes/flipper_1.stl" scale="0.001 0.001 0.001"/></geometry>
     </collision>
     <inertial>
@@ -86,9 +86,9 @@
     <visual>
       <origin rpy="0 0 0" xyz="0.3 0.45 0"/>
-      <geometry><mesh filename="file://$(find aesir_robot_description)/meshes/flipper_2.stl" scale="0.001 0.001 0.001"/></geometry>
+      <geometry><mesh filename="package://aesir_robot_description/meshes/flipper_2.stl" scale="0.001 0.001 0.001"/></geometry>
     </visual>
     <collision>
       <origin rpy="0 0 0" xyz="0.3 0.45 0"/>
-      <geometry><mesh filename="file://$(find aesir_robot_description)/meshes/flipper_2.stl" scale="0.001 0.001 0.001"/></geometry>
+      <geometry><mesh filename="package://aesir_robot_description/meshes/flipper_2.stl" scale="0.001 0.001 0.001"/></geometry>
     </collision>
     <inertial>
@@ -109,9 +109,9 @@
     <visual>
       <origin rpy="0 0 0" xyz="-0.3 1.06 0"/>
-      <geometry><mesh filename="file://$(find aesir_robot_description)/meshes/flipper_3.stl" scale="0.001 0.001 0.001"/></geometry>
+      <geometry><mesh filename="package://aesir_robot_description/meshes/flipper_3.stl" scale="0.001 0.001 0.001"/></geometry>
     </visual>
     <collision>
       <origin rpy="0 0 0" xyz="-0.3 1.06 0"/>
-      <geometry><mesh filename="file://$(find aesir_robot_description)/meshes/flipper_3.stl" scale="0.001 0.001 0.001"/></geometry>
+      <geometry><mesh filename="package://aesir_robot_description/meshes/flipper_3.stl" scale="0.001 0.001 0.001"/></geometry>
     </collision>
     <inertial>
@@ -132,9 +132,9 @@
     <visual>
       <origin rpy="0 0 0" xyz="-0.3 0.45 0"/>
-      <geometry><mesh filename="file://$(find aesir_robot_description)/meshes/flipper_4.stl" scale="0.001 0.001 0.001"/></geometry>
+      <geometry><mesh filename="package://aesir_robot_description/meshes/flipper_4.stl" scale="0.001 0.001 0.001"/></geometry>
     </visual>
     <collision>
       <origin rpy="0 0 0" xyz="-0.3 0.45 0"/>
-      <geometry><mesh filename="file://$(find aesir_robot_description)/meshes/flipper_4.stl" scale="0.001 0.001 0.001"/></geometry>
+      <geometry><mesh filename="package://aesir_robot_description/meshes/flipper_4.stl" scale="0.001 0.001 0.001"/></geometry>
     </collision>
     <inertial>

Commit message: feat(description): upgrade robot base chassis and integrate new sensors description
This major update includes the following structural and visual changes:

- Replaced the old base and flipper meshes with the new tracked chassis files.
- Added accurate 3D meshes for the sensors: LiDAR, and two Logitech C920 cameras (arm and rear).
- Added rescue_robot_v2.urdf.xacro.

File: workspace/src/aesir_robot_description/urdf/rescue_robot.urdf.xacro (robot description, xacro)
@@ -11,4 +11,12 @@
   <xacro:property name="L_TOOL" value="0.28450"/>
   <xacro:property name="L_TOOL_END" value="${L_TOOL-L_WRIST_END}"/>
+  <!-- ============== INITIAL POSITIONS ============== -->
+  <xacro:property name="INIT_J1" value="0.0"/>
+  <xacro:property name="INIT_J2" value="-2.86234"/>
+  <xacro:property name="INIT_J3" value="2.86234"/>
+  <xacro:property name="INIT_J4" value="-1.5708"/>
+  <xacro:property name="INIT_J5" value="-1.5708"/>
+  <xacro:property name="INIT_J6" value="0.0"/>
+  <xacro:property name="INIT_FLIP" value="0.0"/>
   <!-- ================= MATERIALES ================= -->
   <material name="gray"><color rgba="0.7 0.7 0.7 1.0"/></material>
@@ -59,4 +67,99 @@
     </inertial>
   </link>
+  <!-- ================= SENSORS ================= -->
+  <link name="lidar_link">
+    <visual>
+      <origin rpy="0 0 0" xyz="0 0 0"/>
+      <geometry>
+        <mesh filename="package://aesir_robot_description/meshes/lidar.stl" scale="0.001 0.001 0.001"/>
+      </geometry>
+      <material name="black"/>
+    </visual>
+    <collision>
+      <origin rpy="0 0 0" xyz="0 0 0"/>
+      <geometry>
+        <mesh filename="package://aesir_robot_description/meshes/lidar.stl" scale="0.001 0.001 0.001"/>
+      </geometry>
+    </collision>
+    <inertial>
+      <mass value="0.2"/>
+      <inertia ixx="0.001" ixy="0" ixz="0" iyy="0.001" iyz="0" izz="0.001"/>
+    </inertial>
+  </link>
+  <joint name="lidar_joint" type="fixed">
+    <parent link="base_link"/>
+    <child link="lidar_link"/>
+    <origin xyz="0.357 0 0.09" rpy="0 0.785398 0"/>
+  </joint>
+  <link name="oakd_link">
+    <visual>
+      <geometry>
+        <box size="0.02 0.1 0.03"/>
+      </geometry>
+      <material name="gray"/>
+    </visual>
+    <collision>
+      <geometry>
+        <box size="0.02 0.1 0.03"/>
+      </geometry>
+    </collision>
+    <inertial>
+      <mass value="0.1"/>
+      <inertia ixx="0.0001" ixy="0" ixz="0" iyy="0.0001" iyz="0" izz="0.0001"/>
+    </inertial>
+  </link>
+  <joint name="oakd_joint" type="fixed">
+    <parent link="base_link"/>
+    <child link="oakd_link"/>
+    <origin xyz="0.257 0 0.15" rpy="0 0 0"/>
+  </joint>
+  <link name="arm_camera_link">
+    <visual>
+      <origin rpy="0 0 -1.5708" xyz="0 0.05 -0.2"/>
+      <geometry>
+        <mesh filename="package://aesir_robot_description/meshes/logitech_c920.stl" scale="0.001 0.001 0.001"/>
+      </geometry>
+      <material name="black"/>
+    </visual>
+    <collision>
+      <origin rpy="0 0 -1.5708" xyz="0 0.05 -0.2"/>
+      <geometry>
+        <mesh filename="package://aesir_robot_description/meshes/logitech_c920.stl" scale="0.001 0.001 0.001"/>
+      </geometry>
+    </collision>
+    <inertial>
+      <mass value="0.05"/>
+      <inertia ixx="0.00001" ixy="0" ixz="0" iyy="0.00001" iyz="0" izz="0.00001"/>
+    </inertial>
+  </link>
+  <joint name="arm_camera_joint" type="fixed">
+    <parent link="link_6"/>
+    <child link="arm_camera_link"/>
+    <origin xyz="0 -0.03 0.06" rpy="-0.174533 0 0"/>
+  </joint>
+  <link name="back_camera_link">
+    <visual>
+      <origin rpy="0 0 3.14159" xyz="0.04 -0.027 -0.19"/>
+      <geometry>
+        <mesh filename="package://aesir_robot_description/meshes/logitech_c920.stl" scale="0.001 0.001 0.001"/>
+      </geometry>
+      <material name="black"/>
+    </visual>
+    <collision>
+      <origin rpy="0 0 3.14159" xyz="0.04 -0.027 -0.19"/>
+      <geometry>
+        <mesh filename="package://aesir_robot_description/meshes/logitech_c920.stl" scale="0.001 0.001 0.001"/>
+      </geometry>
+    </collision>
+    <inertial>
+      <mass value="0.05"/>
+      <inertia ixx="0.00001" ixy="0" ixz="0" iyy="0.00001" iyz="0" izz="0.00001"/>
+    </inertial>
+  </link>
+  <joint name="back_camera_joint" type="fixed">
+    <parent link="base_link"/>
+    <child link="back_camera_link"/>
+    <origin xyz="-0.35 0 0.1" rpy="0 0 3.14159"/>
+  </joint>
   <!-- ================= FLIPPER 1 ================= -->
   <link name="flipper_1_link">
@@ -321,11 +424,11 @@
   <link name="link_6">
     <visual>
-      <origin xyz="0 ${L_TOOL_END/2} 0" rpy="${-pi/2} 0 0"/>
-      <geometry><cylinder radius="0.01" length="${L_TOOL_END}"/></geometry>
+      <origin xyz="0 0 0" rpy="${-pi/2} 0 0"/>
+      <geometry><cylinder radius="0.01" length="0"/></geometry>
       <material name="orange"/>
     </visual>
     <collision>
-      <origin xyz="0 ${L_TOOL_END/2} 0" rpy="${-pi/2} 0 0"/>
-      <geometry><cylinder radius="0.01" length="${L_TOOL_END}"/></geometry>
+      <origin xyz="0 0 0" rpy="${-pi/2} 0 0"/>
+      <geometry><cylinder radius="0.01" length="0"/></geometry>
     </collision>
     <inertial>
@@ -336,16 +439,80 @@
     </inertial>
   </link>
-  <!-- TOOL -->
-  <joint name="joint_tool" type="fixed">
+    <!-- ================= GRIPPER ================= -->
+  <link name="gripper_base_link">
+    <visual>
+      <origin xyz="0 0.02 0" rpy="0 0 0"/>
+      <geometry>
+        <box size="0.08 0.04 0.06"/>
+      </geometry>
+      <material name="black"/>
+    </visual>
+    <collision>
+      <origin xyz="0 0.02 0" rpy="0 0 0"/>
+      <geometry>
+        <box size="0.08 0.04 0.06"/>
+      </geometry>
+    </collision>
+    <inertial>
+      <mass value="0.3"/>
+      <inertia ixx="0.001" ixy="0" ixz="0" iyy="0.001" iyz="0" izz="0.001"/>
+    </inertial>
+  </link>
+  <joint name="gripper_mount_joint" type="fixed">
     <parent link="link_6"/>
-    <child link="tool_link"/>
-    <origin xyz="0 ${L_TOOL_END} 0" rpy="0 0 0"/>
-  </joint>
-  <link name="tool_link">
-    <visual>
-      <geometry>
-        <box size="0.001 0.001 0.001"/>
-      </geometry>
-    </visual>
-  </link>
+    <child link="gripper_base_link"/>
+    <origin xyz="0 0 0" rpy="0 0 0"/>
+  </joint>
+  <link name="left_finger_link">
+    <visual>
+      <origin xyz="0 0.04 0" rpy="0 0 0"/>
+      <geometry>
+        <box size="0.01 0.08 0.02"/>
+      </geometry>
+      <material name="orange"/>
+    </visual>
+    <collision>
+      <origin xyz="0 0.04 0" rpy="0 0 0"/>
+      <geometry>
+        <box size="0.01 0.08 0.02"/>
+      </geometry>
+    </collision>
+    <inertial>
+      <mass value="0.05"/>
+      <inertia ixx="0.0001" ixy="0" ixz="0" iyy="0.0001" iyz="0" izz="0.0001"/>
+    </inertial>
+  </link>
+  <joint name="left_finger_joint" type="prismatic">
+    <parent link="gripper_base_link"/>
+    <child link="left_finger_link"/>
+    <origin xyz="-0.035 0.04 0" rpy="0 0 0"/>
+    <axis xyz="1 0 0"/>
+    <limit lower="0" upper="0.03" effort="50.0" velocity="0.5"/>
+  </joint>
+  <link name="right_finger_link">
+    <visual>
+      <origin xyz="0 0.04 0" rpy="0 0 0"/>
+      <geometry>
+        <box size="0.01 0.08 0.02"/>
+      </geometry>
+      <material name="orange"/>
+    </visual>
+    <collision>
+      <origin xyz="0 0.04 0" rpy="0 0 0"/>
+      <geometry>
+        <box size="0.01 0.08 0.02"/>
+      </geometry>
+    </collision>
+    <inertial>
+      <mass value="0.05"/>
+      <inertia ixx="0.0001" ixy="0" ixz="0" iyy="0.0001" iyz="0" izz="0.0001"/>
+    </inertial>
+  </link>
+  <joint name="right_finger_joint" type="prismatic">
+    <parent link="gripper_base_link"/>
+    <child link="right_finger_link"/>
+    <origin xyz="0.035 0.04 0" rpy="0 0 0"/>
+    <axis xyz="-1 0 0"/>
+    <limit lower="0" upper="0.03" effort="50.0" velocity="0.5"/>
+  </joint>
 </robot>
